File: Macro_Keyboard_Circuit/Macro_Keyboard_Circuit.kicad_pcb (KiCad board)
At the start: 2 copper layers, 305.2 x 220.2 mm, 55 parts, among them J1 OSTTC082162, J2 PRT-16766, SW1 SW_Push, SW10 SW_Push, SW11 SW_Push, SW12 SW_Push, SW2 SW_Push, SW3 SW_Push, SW4 SW_Push, SW5 SW_Push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

Commit message: Restarting project with new structure
Parts:
- removed LED10, LED11, LED12: HSMW-C280, HSMW_C280:LED_HSMW-C280_BRA
- removed R10, R11, R12: SMD-RES-33R-1_-1_16W_0402_, RC0402FR-0733RL:R0402
- R1, R2, R3, R4, R5, R6, R7, R8, R9: value SMD-RES-33R-1_-1_16W_0402_ -> 33R
- moved R9 116.9 mm to (109.5, 115.5), turned to 180 degrees
- moved LED9 89.4 mm to (112.0, 112.0), turned to 180 degrees
- moved LED8 46.0 mm to (113.0, 172.9), turned to 180 degrees
- moved LED7 36.0 mm to (114.0, 136.5), turned to 180 degrees
- moved R7 31.5 mm to (109.5, 137.0)
- moved J1 31.1 mm to (29.0, 121.2), turned to 90 degrees
- moved R8 23.9 mm to (107.0, 174.0), turned to 90 degrees
- moved U2 18.0 mm to (55.9, 100.4), turned to 0 degrees
- moved J2 1.67 mm to (103.0, 193.6), turned to 0 degrees
Connections:
- J1 pad 7: Net-(U2-G) -> GND
- J2 pad 4: Net-(J2-GND) -> GND
- LED1 pad 1: Net-(J2-GND) -> GND
- LED2 pad 1: Net-(J2-GND) -> GND
- LED3 pad 1: Net-(J2-GND) -> GND
- LED4 pad 1: Net-(J2-GND) -> GND
- LED5 pad 1: Net-(J2-GND) -> GND
- LED6 pad 1: Net-(J2-GND) -> GND
- LED7 pad 1: Net-(J2-GND) -> GND
- LED8 pad 1: Net-(J2-GND) -> GND
- LED9 pad 1: Net-(LED10-Pad1) -> GND
- Layer_SW1 pad 1: Net-(U2-G) -> GND
- Layer_SW1 pad 2: Net-(U2-D2) -> Net-(U2-D0)
- R9 pad 1: Net-(R10-Pad1) -> Net-(J2-3V)
- U1 pad CLK: Net-(J2-D12) -> Net-(J2-D13)
- U1 pad DT: Net-(J2-D13) -> Net-(J2-D12)
- U1 pad GND: Net-(U2-G) -> GND
- U2 pad 10: Net-(U2-MISO) -> /Col2
- U2 pad 12: Net-(U2-D10) -> /Col1
- U2 pad 13: /Col1 -> /Col3
- U2 pad 14: /Col2 -> /Col4
- U2 pad 15: /Col3 -> Net-(U2-D7)
- U2 pad 16: /Col4 -> Net-(U2-D6)
- U2 pad 17: /Row3 -> /Row1
- U2 pad 19: /Row1 -> /Row3
- U2 pad 2: Net-(U2-G) -> GND
- U2 pad 21: unconnected-(U2-GND-Pad21) -> GND
- U2 pad 22: unconnected-(U2-GND-Pad22) -> GND
- U3 pad CLK: Net-(U2-D10) -> Net-(U2-D2)
- U3 pad DT: Net-(U2-MISO) -> Net-(U2-D1)
- U3 pad GND: Net-(U2-G) -> unconnected-(U3-PadGND)
- U4 pad CLK: Net-(U2-D1) -> Net-(U2-D7)
- U4 pad DT: Net-(U2-D0) -> Net-(U2-D6)
- U4 pad GND: Net-(U2-G) -> GND
Routing:
- net Net-(J2-GND): track 193.5 -> 0.00 mm, vias 2 -> 0
- net Net-(U2-G): track 168.4 -> 0.00 mm
- net Net-(U2-D10): track 92.6 -> 0.00 mm
- net Net-(U2-MISO): track 86.6 -> 0.00 mm
- net /Row1: track 85.7 -> 172.2 mm
- net Net-(U2-D7): track 0.00 -> 81.0 mm, vias 0 -> 1
- net Net-(U2-D6): track 0.00 -> 81.0 mm, vias 0 -> 1
- net Net-(U2-RAW_(5V)): track 182.3 -> 232.2 mm
- net /Row2: track 119.6 -> 164.6 mm
- net Net-(J2-3V): track 158.0 -> 201.1 mm
- net Net-(U2-D0): track 79.2 -> 50.8 mm
- net /Col4: track 98.0 -> 72.9 mm
- net /Col3: track 81.3 -> 61.0 mm
- net /Row3: track 143.6 -> 163.5 mm
- net Net-(U2-D2): track 79.4 -> 60.3 mm
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- added copper zone on B.Cu, net GND
- added copper zone on F.Cu, net GND
Other:
- board size 305.2 x 220.2 mm -> 115.2 x 117.1 mm
