File: Macro_Keyboard_Circuit/Macro_Keyboard_Circuit.kicad_sch (KiCad schematic)
At the start: 55 parts, among them J1 OSTTC082162, J2 PRT-16766, SW1 SW_Push, SW10 SW_Push, SW11 SW_Push, SW12 SW_Push, SW2 SW_Push, SW3 SW_Push, SW4 SW_Push, SW5 SW_Push, SW6 SW_Push, SW7 SW_Push, SW8 SW_Push, SW9 SW_Push, U1 KY-040, U2 Adafruit KB2040, U3 KY-040, U4 KY-040

Commit message: Restarting project with new structure
Parts:
- removed LED10, LED11, LED12: HSMW-C280, HSMW_C280:LED_HSMW-C280_BRA, symbol HSMW_C280:HSMW-C280
- removed R10, R11, R12: SMD-RES-33R-1_-1_16W_0402_, RC0402FR-0733RL:R0402, symbol RC0402FR-0733RL:SMD-RES-33R-1_-1_16W_0402_
- R1, R2, R3, R4, R5, R6, R7, R8, R9: value SMD-RES-33R-1_-1_16W_0402_ -> 33R; VALUE 33R -> (none)
Connections:
- net Col1: now also U2.12 (D10); no longer U2.13 (D9)
- net Col2: now also U2.10 (MISO); no longer U2.14 (D8)
- net Col3: now also U2.13 (D9); no longer U2.15 (D7)
- net Col4: now also U2.14 (D8); no longer U2.16 (D6)
- net GND: now also J1.7, J2.4 (GND), LED1.1, LED2.1, LED3.1, LED4.1, LED5.1, LED6.1, LED7.1, LED8.1, LED9.1, Layer_SW1.1, U1.GND, U2.2 (G), U2.21 (GND), U2.22 (GND), U4.GND
- net Row1: now also U2.17 (D5); no longer U2.19 (D3)
- net Row3: now also U2.19 (D3); no longer U2.17 (D5)
- net at J2.3 (3V), R1.1, R2.1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: now also R9.1
- net at U1.CLK: now also J2.1 (D13); no longer J2.2 (D12)
- net at U1.DT: now also J2.2 (D12); no longer J2.1 (D13)
- net at U3.DT: now also U2.23 (D1); no longer U2.10 (MISO)
- net at U3.CLK: now also U2.20 (D2); no longer U2.12 (D10)
- net at Layer_SW1.2: now also U2.24 (D0); no longer U2.20 (D2)
- net at U4.CLK: now also U2.15 (D7); no longer U2.23 (D1)
- net at U4.DT: now also U2.16 (D6); no longer U2.24 (D0)
- now unconnected: U3.GND
Other:
- moved on the sheet: J1, Layer_SW1, U3, U4
